Commit message: mtc and final project

File: xarm_moveit_config/srdf/_xarm6_macro.srdf.xacro (robot description, xacro)
@@ -73,4 +73,7 @@
       <group_state name="close" group="${prefix}xarm_gripper">
         <joint name="${prefix}drive_joint" value="0.85" />
+      </group_state>
+      <group_state name="grasp" group="${prefix}xarm_gripper">
+        <joint name="${prefix}drive_joint" value="0.5" />
       </group_state>
       <!-- END EFFECTOR, Purpose, Represent information about an end effector. -->
